File: sensor_node.kicad_pcb (KiCad board)
At the start: 2 copper layers, 80 x 30 mm, 88 parts, among them J1 Conn_01x06_Male, J10 Conn_01x06, J11 Conn_02x08_Counter_Clockwise, J2 Conn_01x03, J3 USB_B_Micro, J4 Conn_01x02_Female, J5 Conn_01x08_Male, J6 Conn_01x04_Male, J7 Conn_Coaxial, J8 Conn_02x04_Odd_Even, Q5 Q_PMOS_GSD, Q6 Q_PMOS_GSD, Q7 Q_PMOS_GSD, U1 STM32L063R8Tx, U3 BME680, U4 Si1133, U5 USBLC6-2SC6, U7 BQ24075, U8 TPS826711, U9 LMZ21700, Y1 Crystal_GND24

Commit message: worked on board
Parts:
- removed C30, C31: 10uF, Capacitor_SMD:C_0805_2012Metric_Pad1.15x1.40mm_HandSolder
- added J9: Conn_01x03, Connector_JST:JST_EH_S3B-EH_1x03_P2.50mm_Horizontal, F.Cu at (106.6, 92.6)
- C1, C2, C34, C35, C4, C5, C8, J8, R3, Y1: moved to B.Cu
- J6: footprint Connector_PinHeader_2.54mm:PinHeader_1x04_P2.54mm_Vertical -> Connector_PinHeader_2.54mm:PinHeader_1x04_P2.54mm_Horizontal
- moved J11 72.5 mm to (147.6, 77.0)
- moved J6 56.4 mm to (79.4, 114.6), turned to 270 degrees
- moved Y1 53.8 mm to (69.8, 91.6), turned to 270 degrees
- moved C8 51.4 mm to (72.8, 92.8), turned to 270 degrees
- moved C5 49.4 mm to (72.8, 90.2), turned to 90 degrees
- moved J8 46.0 mm to (112.6, 117.4), turned to 90 degrees
- moved J5 40.6 mm to (99.0, 77.0), turned to 0 degrees
- moved C1 34.3 mm to (74.0, 87.1), turned to 90 degrees
- moved Q7 31.8 mm to (142.4, 93.4)
- moved C34 30.8 mm to (73.2, 78.0), turned to 90 degrees
- moved J2 30.6 mm to (93.1, 92.6), turned to 180 degrees
- moved R13 28.3 mm to (92.1, 89.8), turned to 0 degrees
- moved C35 26.6 mm to (70.6, 77.2), turned to 180 degrees
- moved C10 24.2 mm to (88.0, 97.4)
- moved R10 21.8 mm to (82.6, 101.9), turned to 90 degrees
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Connections:
- net /mcu.sch/PA10 renamed /DSIP_BUSY
- net /mcu.sch/PA6 renamed /SPI1_MISO
- C17 pad 1: /power_supply/VUSB -> /VUSB
- C19 pad 1: /power_supply/VUSB -> /VUSB
- C3 pad 1: /power_supply/VUSB -> /VUSB
- FB2 pad 1: /power_supply/VUSB -> /VUSB
- R3 pad 1: /mcu.sch/VUSB -> /VUSB
- U1 pad 21: /mcu.sch/PA5 -> /SPI1_SCK
- U1 pad 23: /mcu.sch/PA7 -> /SPI1_MOSI
- U1 pad 41: /mcu.sch/PA8 -> /DISP_DC
- U1 pad 42: /mcu.sch/PA9 -> /DISP_RST
- U5 pad 4: /power_supply/USB_DN -> /mcu.sch/PA11
- U5 pad 5: /power_supply/VUSB -> /VUSB
- U5 pad 6: /power_supply/USB_DP -> /mcu.sch/PA12
- U7 pad 13: /power_supply/VUSB -> /VUSB

Commit message: further work
Parts:
- added C16: 10uF, Capacitor_SMD:C_0603_1608Metric, F.Cu at (131.8, 59.3)
- added C18: 100nF, Capacitor_SMD:C_0603_1608Metric, F.Cu at (125.5, 67.9)
- added C30: 10uF, Capacitor_SMD:C_0603_1608Metric_Pad1.05x0.95mm_HandSolder, F.Cu at (116.9, 65.3)
- added C31: 100nF, Capacitor_SMD:C_0603_1608Metric_Pad1.05x0.95mm_HandSolder, F.Cu at (121.3, 65.3)
- added C32: 2.2pf,25V, Capacitor_SMD:C_0603_1608Metric_Pad1.05x0.95mm_HandSolder, F.Cu at (116.9, 67.9)
- added C33: 10uF, Capacitor_SMD:C_0603_1608Metric_Pad1.05x0.95mm_HandSolder, F.Cu at (127.6, 59.3)
- added C36: 100nF, Capacitor_SMD:C_0603_1608Metric_Pad1.05x0.95mm_HandSolder, F.Cu at (121.3, 67.9)
- added J13: Conn_Coaxial, Connector_Coaxial:U.FL_Hirose_U.FL-R-SMT-1_Vertical, F.Cu at (117.3, 61.1)
- added J14: Conn_Coaxial, Connector_Coaxial:U.FL_Hirose_U.FL-R-SMT-1_Vertical, F.Cu at (122.6, 61.1)
- added L1: 8.2nH,2%, Inductor_SMD:L_0603_1608Metric_Pad1.05x0.95mm_HandSolder, F.Cu at (125.6, 65.3)
- added Q1: Q_NMOS_GSD, Package_TO_SOT_SMD:SOT-23_Handsoldering, F.Cu at (109.4, 61.3)
- added R11: R, Resistor_SMD:R_0603_1608Metric_Pad1.05x0.95mm_HandSolder, F.Cu at (127.6, 61.8)
- added U2: NEO-M8Q, RF_GPS:ublox_NEO, F.Cu at (98.5, 67.8)

Commit message: add docu
more changes
Parts:
- removed J11: Conn_02x08_Counter_Clockwise, Connector_PinHeader_2.54mm:PinHeader_2x08_P2.54mm_Vertical_SMD
- removed J7: Conn_Coaxial, Connector_Coaxial:U.FL_Hirose_U.FL-R-SMT-1_Vertical
- removed JP5: SolderJumper_3_Bridged12, Jumper:SolderJumper-3_P1.3mm_Bridged12_RoundedPad1.0x1.5mm
- removed R28: 10k, Resistor_SMD:R_0603_1608Metric_Pad1.05x0.95mm_HandSolder
- removed R29: 147k, Resistor_SMD:R_0603_1608Metric_Pad1.05x0.95mm_HandSolder
- removed R30: 118k, Resistor_SMD:R_0603_1608Metric_Pad1.05x0.95mm_HandSolder
- added AE1: Antenna_Chip, RF_Antenna:0868AT43A0020, F.Cu at (122.2, 92.4)
- added H1: MountingHole_Pad, MountingHole:MountingHole_3.5mm_Pad, F.Cu at (126.2, 73.6)
- added H2: MountingHole_Pad, MountingHole:MountingHole_3.5mm_Pad, F.Cu at (54.3, 74.2)
- added H3: MountingHole_Pad, MountingHole:MountingHole_3.5mm_Pad, F.Cu at (54.6, 95.4)
- added JP6: SolderJumper_2_Open, Jumper:SolderJumper-2_P1.3mm_Open_RoundedPad1.0x1.5mm, F.Cu at (116.0, 85.9)
- added L2: 18nH, Inductor_SMD:L_0603_1608Metric, F.Cu at (117.0, 90.3)
- added Q2: Q_NMOS_DGS, Package_TO_SOT_SMD:SOT-23_Handsoldering, B.Cu at (88.2, 88.3)
- added Q3: Q_NMOS_DGS, Package_TO_SOT_SMD:SOT-23_Handsoldering, F.Cu at (108.2, 73.8)
- added R12: R_Small, Resistor_SMD:R_0603_1608Metric_Pad1.05x0.95mm_HandSolder, B.Cu at (83.4, 85.1)
- added R17: 4.7k, Resistor_SMD:R_0603_1608Metric_Pad1.05x0.95mm_HandSolder, B.Cu at (61.1, 84.2)
- added R18: R_Small, Resistor_SMD:R_0603_1608Metric_Pad1.05x0.95mm_HandSolder, F.Cu at (114.8, 72.8)
- added U10: E78-868LN22S, RF_Module:e22-868ln22s, F.Cu at (99.5, 89.5)
- C10, C11, C12, C16, C18, C30, C31, C33, C36, C7, C9, FB1, Q1, Q6, R1, R11, U2: moved to B.Cu
- C13, C14, C15, JP1, U3, U4: moved to F.Cu
- C22: value C -> 1uF; footprint Capacitor_SMD:C_0805_2012Metric_Pad1.15x1.40mm_HandSolder -> Capacitor_SMD:C_0603_1608Metric_Pad1.05x0.95mm_HandSolder
- C23: value C -> 1uF
- C24: value CP -> 1uF; footprint Capacitor_SMD:C_0805_2012Metric_Pad1.15x1.40mm_HandSolder -> Capacitor_SMD:C_0603_1608Metric_Pad1.05x0.95mm_HandSolder
- C25: value 22uF -> 1uF; footprint Capacitor_SMD:C_0805_2012Metric_Pad1.15x1.40mm_HandSolder -> Capacitor_SMD:C_0603_1608Metric_Pad1.05x0.95mm_HandSolder
- C26: value 3300pF -> 3.9pF; footprint Capacitor_SMD:C_0603_1608Metric_Pad1.05x0.95mm_HandSolder -> Capacitor_SMD:C_0603_1608Metric; moved to F.Cu
- C27: value 22uF -> 0.3pF; footprint Capacitor_SMD:C_0805_2012Metric_Pad1.15x1.40mm_HandSolder -> Capacitor_SMD:C_0603_1608Metric; moved to F.Cu
- J4: footprint Connector_JST:JST_EH_S2B-EH_1x02_P2.50mm_Horizontal -> Connector_JST:JST_EH_B2B-EH-A_1x02_P2.50mm_Vertical; moved to F.Cu
- J6: footprint Connector_PinHeader_2.54mm:PinHeader_1x04_P2.54mm_Horizontal -> Connector_PinHeader_2.54mm:PinHeader_1x04_P2.54mm_Vertical
- J8: footprint Connector_PinHeader_2.54mm:PinHeader_2x04_P2.54mm_Vertical -> Connector_PinHeader_2.54mm:PinHeader_2x04_P2.54mm_Vertical_SMD
- U8: value TPS826711 -> LD39015M33R; footprint Package_CSP:Texas_SIP0009F_MicroSiP-8_2.3x2.9mm_P0.8mm -> Package_TO_SOT_SMD:SOT-23-5
- U9: value LMZ21700 -> LD39015M18R; footprint Package_LGA:Texas_SIL0008E_MicroSip-8-2EP_3.5x3.5mm_P0.8mm_EP0.8x1.9mm -> Package_TO_SOT_SMD:SOT-23-5
- moved C11 64.6 mm to (110.9, 73.3), turned to 180 degrees
- moved C12 63.6 mm to (110.9, 71.5), turned to 180 degrees
- moved J10 58.3 mm to (70.7, 97.1), turned to 90 degrees
- moved Q5 55.7 mm to (111.8, 73.8), turned to 90 degrees
- moved C26 52.9 mm to (116.2, 88.0)
- moved C27 50.6 mm to (116.2, 92.6)
- moved R11 50.3 mm to (89.7, 94.9)
- moved R10 45.3 mm to (39.4, 115.8)
- moved C9 45.2 mm to (82.3, 75.1), turned to 180 degrees
- moved R1 43.9 mm to (70.0, 86.1), turned to 270 degrees
- moved J6 42.6 mm to (78.5, 72.0), turned to 90 degrees
- moved C33 42.6 mm to (109.6, 97.9), turned to 90 degrees
- moved J8 42.4 mm to (117.2, 75.3), turned to 180 degrees
- moved J9 42.0 mm to (142.7, 71.2), turned to 270 degrees
- moved Q1 37.3 mm to (88.0, 91.9)
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Connections:
- C16 pad 1: /sensors/gps/VCC_3V3 -> /sensors/gps/GPS_VBCK
- C18 pad 1: /sensors/gps/VCC_3V3 -> /sensors/gps/GPS_VBCK
- C21 pad 1: VIN -> /VCC
- C22 pad 1: VIN -> /VCC
- C23 pad 1: VIN -> /VCC
- C24 pad 1: /VCC_1V8 -> /VCC_3V3
- C25 pad 1: VIN -> /VCC_1V8
- C27 pad 1: /VCC_3V3 -> Net-(AE1-Pad1)
- C30 pad 1: /sensors/gps/VBCKP -> /sensors/gps/GPS_VBCK
- C31 pad 1: /sensors/gps/VBCKP -> /sensors/gps/GPS_VBCK
- D4 pad 2: /mcu.sch/PA0 -> /mcu.sch/PA1
- J10 pad 1: /VCC_3V3 -> /PC3
- J10 pad 2: /PC3 -> /PC4
- J10 pad 4: /PC4 -> /PC5
- J10 pad 5: /PC5 -> /sensor_connectors/EXT_GPIO4
- J10 pad 6: GND -> /sensor_connectors/EXT_GPIO5
- J13 pad 1: Net-(J13-Pad1) -> /sensors/GPS_TIMEPULSE
- J6 pad 2: /I2C1_SDA -> /GPS_SDA
- J6 pad 4: /I2C1_SCL -> /GPS_SCL
- JP3 pad 2: VIN -> /VCC
- Q1 pad 1: Net-(Q1-Pad1) -> /PC15
- Q5 pad 1: /PB2 -> Net-(Q3-Pad1)
- Q5 pad 3: /VCC_1V8 -> /VCC_3V3
- Q6 pad 1: /PC14 -> Net-(Q2-Pad1)
- Q6 pad 3: /sensors/VGPS -> /sensors/gps/GPS_VBCK
- R11 pad 1: /sensors/gps/VCC_3V3 -> Net-(Q1-Pad3)
- R11 pad 2: Net-(Q1-Pad3) -> /sensors/gps/GPS_VBCK
- R2 pad 1: /I2C1_SCL -> /GPS_SCL
- R5 pad 1: /I2C1_SDA -> /GPS_SDA
- U1 pad 16: /EXP_RX -> /LORA_TX
- U1 pad 17: /ESP_TX -> /LORA_RX
- U1 pad 51: /mcu.sch/PC10 -> /ESP_RX
- U1 pad 52: /mcu.sch/PC11 -> /ESP_TX
- U1 pad 58: /STM_PB6 -> /GPS_RX
- U1 pad 59: /STM_PB7 -> /GPS_TX
- U1 pad 61: /I2C1_SCL -> /GPS_SCL
- U1 pad 62: /I2C1_SDA -> /GPS_SDA
- U2 pad 18: /sensors/gps/I2C_SENSOR_SDA -> /GPS_SDA
- U2 pad 19: /sensors/gps/I2C_SENSOR_SCL -> /GPS_SCL
- U2 pad 20: /sensors/gps/GPS_TX -> /GPS_TX
- U2 pad 21: /sensors/gps/GPS_RX -> /GPS_RX
- U2 pad 22: /sensors/gps/VBCKP -> /sensors/gps/GPS_VBCK
- U2 pad 23: /sensors/gps/VGPS -> /sensors/gps/GPS_VBCK
- U2 pad 3: Net-(J13-Pad1) -> /sensors/GPS_TIMEPULSE
- U7 pad 10: VIN -> /VCC
- U7 pad 11: VIN -> /VCC
- U7 pad 5: VIN -> /VCC
- U8 pad 1: /VCC_1V8 -> /VCC
- U8 pad 2: VIN -> GND
- U8 pad 3: VIN -> /EN_3V3
- U8 pad 4: VIN -> Net-(U8-Pad4)
- U8 pad 5: /power_supply/MODE_1V8 -> /VCC_3V3
- U9 pad 1: Net-(C26-Pad1) -> /VCC
- U9 pad 2: Net-(R29-Pad2) -> GND
- U9 pad 3: Net-(R28-Pad2) -> /VCC
- U9 pad 4: /VCC_3V3 -> Net-(U9-Pad4)
- U9 pad 5: GND -> /VCC_1V8
Routing:
- net VIN: track 4.93 -> 0.00 mm
- net /VCC_1V8: track 2.37 -> 0.00 mm
- added copper zone on F.Cu, net Net-(AE1-Pad2)
Other:
- rule trace_min: 0.2 -> 0.1
